File: HW_TestDrive/Clouds.kicad_sch (KiCad schematic)
At the start: 11 parts, among them J1 Conn_01x10, J2 Conn_01x04, U1 AS5600L-ASOM, U2 DRV8313PWPR

Commit message: Revise schematic
Parts:
- added D1: White, LED_SMD:LED_0805_2012Metric, symbol Device:LED
- added D2: Yellow, LED_SMD:LED_0805_2012Metric, symbol Device:LED
- added R3: 2.2k, Resistor_SMD:R_0603_1608Metric, symbol Device:R
- added R4: 1k, Resistor_SMD:R_0603_1608Metric, symbol Device:R
- C1, C2, C3, C4: footprint (none) -> Capacitor_SMD:C_0603_1608Metric
- C5: footprint (none) -> Capacitor_SMD:CP_Elec_5x3.9
- J1: footprint (none) -> Connector_PinHeader_2.54mm:PinHeader_1x10_P2.54mm_Vertical
- J2: footprint (none) -> Connector_PinHeader_2.54mm:PinHeader_1x04_P2.54mm_Vertical
- R1, R2: footprint (none) -> Resistor_SMD:R_0603_1608Metric
Connections:
- net +3.3V: now also R3.1
- net GND: now also D1.1 (K), D2.1 (K)
- net NFAULT: now also R4.1; no longer J2.4 (Pin_4)
- new net: D2.2 (A), R4.2
- new net: D1.2 (A), R3.2
- no-connect marks 5 -> 6

Commit message: (WIP) PCB layout
Parts:
- removed J2: Conn_01x04, Connector_PinHeader_2.54mm:PinHeader_1x04_P2.54mm_Vertical, symbol Connector_Generic:Conn_01x04
- added J2: Conn_01x03, Connector_PinHeader_2.54mm:PinHeader_1x03_P2.54mm_Vertical, symbol Connector_Generic:Conn_01x03
Connections:
- net MOTOR_U: now also J2.1 (Pin_1)
- net MOTOR_V: now also J2.2 (Pin_2)
- net MOTOR_W: now also J2.3 (Pin_3)
- net VCC renamed VM
- no-connect marks 6 -> 5
Changed lines of the file:
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@@
   (no_connect (at 99.06 45.085))
   (no_connect (at 68.58 42.545))
-  (no_connect (at 34.925 70.485))
   (no_connect (at 175.26 61.595))
   (no_connect (at 210.82 53.975))
@@
         (path "/503c6fae-2261-4b98-b430-844cd1712448"
           (reference "#PWR020") (unit 1)
+        )
+      )
+    )
+  )
+  (symbol (lib_id "Connector_Generic:Conn_01x03") (at 29.845 65.405 0) (mirror y) (unit 1)
+    (in_bom yes) (on_board yes) (dnp no) (fields_autoplaced)
+    (property "Reference" "J2" (at 29.845 57.15 0)
+      (effects (font (size 1.27 1.27)))
+    )
+    (property "Value" "Conn_01x03" (at 29.845 59.69 0)
+      (effects (font (size 1.27 1.27)))
+    )
+    (property "Footprint" "Connector_PinHeader_2.54mm:PinHeader_1x03_P2.54mm_Vertical" (at 29.845 65.405 0)
+      (effects (font (size 1.27 1.27)) hide)
+    )
+    (property "Datasheet" "~" (at 29.845 65.405 0)
+      (effects (font (size 1.27 1.27)) hide)
+    )
+    (pin "2")
+    (pin "3")
+    (pin "1")
+    (instances
+      (project "Clouds"
+        (path "/503c6fae-2261-4b98-b430-844cd1712448"
+          (reference "J2") (unit 1)
         )
       )
@@
         )
       )
-    )
-  )
-  (symbol (lib_id "Connector_Generic:Conn_01x04") (at 29.845 65.405 0) (mirror y) (unit 1)
-    (in_bom yes) (on_board yes) (dnp no) (fields_autoplaced)
-    (property "Reference" "J2" (at 29.845 56.515 0)
-      (effects (font (size 1.27 1.27)))
-    )
-    (property "Value" "Conn_01x04" (at 29.845 59.055 0)
-      (effects (font (size 1.27 1.27)))
-    )
-    (property "Footprint" "Connector_PinHeader_2.54mm:PinHeader_1x04_P2.54mm_Vertical" (at 29.845 65.405 0)
-      (effects (font (size 1.27 1.27)) hide)
-    )
-    (property "Datasheet" "~" (at 29.845 65.405 0)
-      (effects (font (size 1.27 1.27)) hide)
-    )
-    (pin "2")
-    (pin "4")
-    (pin "3")
-    (pin "1")
-    (instances
-      (project "Clouds"
-        (path "/503c6fae-2261-4b98-b430-844cd1712448"
-          (reference "J2") (unit 1)
-        )
-      )
