File: HW_TestDrive/Clouds.kicad_pcb (KiCad board)
At the start: 2 copper layers, 21.3 x 26.5 mm, 15 parts, among them J1 Conn_01x10, J2 Conn_01x03, U1 AS5600L-ASOM, U2 DRV8313PWPR

Commit message: (WIP) Almost-complete layout
Parts:
- added G***: LOGO, LOGO, F.Cu at (37.4, 26.7)
- moved C2 2.12 mm to (34.7, 42.6)
- moved C4 1.63 mm to (32.6, 42.6)
Routing:
- net EN_U: track 0.00 -> 12.1 mm
- net Net-(U2-CPH): track 0.00 -> 10.6 mm
- net IN_U: track 0.00 -> 10.1 mm
- net MOTOR_W: track 0.00 -> 8.53 mm
- net EN_V: track 0.00 -> 8.24 mm
- net MOTOR_V: track 0.00 -> 7.61 mm
- net MOTOR_U: track 0.00 -> 7.25 mm
- net IN_V: track 0.00 -> 6.42 mm
- net EN_W: track 0.00 -> 5.64 mm
- net IN_W: track 0.00 -> 4.87 mm
- net GND: track 2.25 -> 6.94 mm, vias 0 -> 32
- net Net-(U2-CPL): track 0.00 -> 4.52 mm
- net Net-(U2-VCP): track 0.00 -> 2.54 mm
- net VM: vias 0 -> 23
- added copper zone on B.Cu, net GND
- added copper zone on F.Cu, net GND
- added copper zone on B.Cu, net VM
- added copper zone on F.Cu, net VM
Other:
- board text added: "*"
- board text added: "23-Flurry"
- board text added: "3-phase BLDC Driver Magnet Encoder Input 8-60 V Output 1.75 A RMS"
- board text added: "BLDC on Clouds"
- board text added: "Rev. 1"

Commit message: Finish PCB design
Parts:
- added G***: LOGO, LOGO, B.Cu at (31.5, 34.9)
- added G***: LOGO, LOGO, B.Cu at (23.8, 33.3)
- added G***: LOGO, LOGO, B.Cu at (28.3, 33.6)
- moved C2 0.48 mm to (34.2, 42.6)
- moved C4 0.48 mm to (32.1, 42.6)
- moved U2 0.48 mm to (27.3, 39.3)
- moved C5 0.30 mm to (34.5, 32.9)
- moved C3 0.20 mm to (26.4, 33.3)
Routing:
- net +3.3V: track 18.5 -> 17.7 mm
- net GND: vias 32 -> 31
Other:
- board text added: "BLDC Driver (Y-wired) Magnet Encoder"
- board text added: "Input 8-60 V Output 1.75 A RMS"
- board text added: "JLCJLCJLCJLC"
- board text removed: "3-phase BLDC Driver Magnet Encoder Input 8-60 V Output 1.75 A RMS"
